File: files/heli_hardware_files/heli_hardware_files.kicad_sch (KiCad schematic)
At the start: 22 parts, among them J1 USB_C_Receptacle_USB2.0_14P, Q1 AO3401A, U2 MPU-6050, U4 SPX3819M5-L-3-3

Commit message: Pcb was added.
Parts:
- added C10: 10uF, Capacitor_SMD:C_0603_1608Metric, symbol Device:C
- added C11, C9: 100nF, Capacitor_SMD:C_0603_1608Metric, symbol Device:C
- added R9: 4.7k, Resistor_SMD:R_0603_1608Metric, symbol Device:R
- added U1: ESP32-S3-WROOM-1-N8, ESP32-S3-WROOM-1-N8:XCVR_ESP32-S3-WROOM-1-N8, symbol ESP32-S3-WROOM-1-N8:ESP32-S3-WROOM-1-N8
- C1, C2, C3, C4, C5, C6, C7, C8: footprint (none) -> Capacitor_SMD:C_0603_1608Metric
- R1, R2, R3, R4, R5, R6, R7, R8: footprint (none) -> Resistor_SMD:R_0603_1608Metric
Connections:
- net +3.3V: now also C10.2, C11.2, R9.1, U1.2 (3V3)
- net GND: now also C10.1, C11.1, C9.1, U1.1 (GND), U1.40 (GND), U1.41_1 (GND), U1.41_2 (GND), U1.41_3 (GND), U1.41_4 (GND), U1.41_5 (GND), U1.41_6 (GND), U1.41_7 (GND), U1.41_8 (GND), U1.41_9 (GND)
- new net EN: C9.2, R9.2, U1.3 (EN)
- no-connect marks 2 -> 0
